Commit message: feat: add rear caster wheel and rviz config for SLAM

File: Prodev_simulation/urdf/robot.urdf (robot description, URDF)
Before this commit: robot robot, 8 links, 7 joints
Links:
- added link rear_caster_link, mass 0.1; collision sphere radius=0.02; visual sphere radius=0.02
Joints:
- added joint rear_caster_joint: type fixed, parent base_link, child rear_caster_link, origin xyz=-0.12 0 -0.03 rpy=0 0 0

Commit message: fix(Prodev_simulation): colocate IMU frame with base_link for Cartographer

File: Prodev_simulation/urdf/robot.urdf (robot description, URDF)
Before this commit: robot robot, 9 links, 8 joints
Joints:
- joint imu_joint: origin xyz=0 0 0.02 rpy=0 0 0 -> xyz=0 0 0.0 rpy=0 0 0
